File: EasyDroidVR_PCB/EasyDroidVR_PCB.kicad_sch (KiCad schematic)
At the start: 37 parts, among them J1 PINHD_1x12_Male, J10 PINHD_1x1_Male, J11 PINHD_1x1_Male, J12 PINHD_1x1_Male, J13 PINHD_1x1_Male, J14 PINHD_1x1_Male, J2 PINHD_1x12_Male, J3 MPU6500, J4 Battery Holder -, J5 Battery Holder +, J6 JST_09, J7 PINHD_1x1_Male, J8 PINHD_1x1_Male, J9 PINHD_1x1_Male, Q1 2N7000, Q4 2N7000, Q5 2N7000, Q6 2N7000, Q7 2N7000, Q8 2N7000, U1 NRF24L01_Breakout, U6 COM-09032

Commit message: V1.0 Working
Parts:
- removed D2: WS2812B, LED_SMD:LED_WS2812B_PLCC4_5.0x5.0mm_P3.2mm, symbol LED:WS2812B
- removed J1, J2: PINHD_1x12_Male, Connector_PinHeader_2.54mm:PinHeader_1x12_P2.54mm_Vertical, symbol PCM_SL_Pin_Headers:PINHD_1x12_Male
- removed J10, J13, J7, J8, J9: PINHD_1x1_Male, Connector_PinHeader_2.54mm:PinHeader_1x01_P2.54mm_Vertical, symbol PCM_SL_Pin_Headers:PINHD_1x1_Male
- removed J5: Battery Holder +, Connector_PinSocket_2.54mm:PinSocket_1x01_P2.54mm_Vertical, symbol PCM_SL_Pin_Headers:PINHD_1x1_Female
- removed J6: JST_09, Connector_JST:JST_EH_B9B-EH-A_1x09_P2.50mm_Vertical, symbol PCM_SL_Connectors:JST_09
- removed Q1, Q4, Q5, Q6, Q7, Q8: 2N7000, PCM_Package_TO_SOT_THT_AKL:TO-92_Inline_Wide_SGD, symbol PCM_Transistor_MOSFET_AKL:2N7000
- removed R1, R10, R11, R12, R13, R14, R15, R2, R6, R7, R8, R9: R_1210 4.7KOhm, PCM_Resistor_SMD_AKL:R_1210_3225Metric, symbol PCM_Resistor_AKL:R_1210
- removed R16: R_1210 330Ohm, PCM_Resistor_SMD_AKL:R_1210_3225Metric, symbol PCM_Resistor_AKL:R_1210
- removed U6: COM-09032, COM-09032:XDCR_COM-09032, symbol COM-09032:COM-09032
- added A1: STM32_Blue_Pill_DevBoard, PCM_SL_Development_Boards:STM32_Blue_Pill_DevBoard, symbol PCM_SL_Development_Board:STM32_Blue_Pill_DevBoard
- added C1, C2, C4: 100nF_Ceramic, Capacitor_THT:C_Disc_D5.0mm_W2.5mm_P2.50mm, symbol PCM_SL_Capacitors:100nF_Ceramic
- added C10, C9: C_0603 20pF, PCM_Capacitor_SMD_AKL:C_0603_1608Metric, symbol PCM_Capacitor_AKL:C_0603
- added C11, C12, C13, C14, C15: C_0603 100nF, PCM_Capacitor_SMD_AKL:C_0603_1608Metric, symbol PCM_Capacitor_AKL:C_0603
- added C3: 470uF_16V, Capacitor_THT:CP_Radial_D8.0mm_P3.50mm, symbol PCM_SL_Capacitors:470uF_16V
- added C6: 100uF_10V, Capacitor_THT:CP_Radial_D5.0mm_P2.00mm, symbol PCM_SL_Capacitors:100uF_10V
- added C7: 47uF_10V, Capacitor_THT:CP_Radial_D4.0mm_P1.50mm, symbol PCM_SL_Capacitors:47uF_10V
- added C8: 10nF_Ceramic, Capacitor_THT:C_Disc_D5.0mm_W2.5mm_P2.50mm, symbol PCM_SL_Capacitors:10nF_Ceramic
- added D2: LED_3mm, LED_THT:LED_D3.0mm, symbol PCM_SL_Devices:LED_3mm
- added H1, H2, H3, H4: MountingHole_M3, MountingHole:MountingHole_3.2mm_M3, symbol PCM_SL_Mechanical:MountingHole_M3
- added J1: PINHD_1x2_Female, Battery:BatteryHolder_MYOUNG_BS-07-A1BJ001_CR2032, symbol PCM_SL_Pin_Headers:PINHD_1x2_Female
- added J13: PINHD_1x5_Female Joystick, Connector_PinSocket_2.54mm:PinSocket_1x05_P2.54mm_Vertical, symbol PCM_SL_Pin_Headers:PINHD_1x5_Female
- added J15, J16: PINHD_1x1_Male, TestPoint:TestPoint_THTPad_2.0x2.0mm_Drill1.0mm, symbol PCM_SL_Pin_Headers:PINHD_1x1_Male
- added J2: PINHD_1x5_Female, Connector_PinSocket_2.54mm:PinSocket_1x05_P2.54mm_Vertical, symbol PCM_SL_Pin_Headers:PINHD_1x5_Female
- added J6: PINHD_1x5_Male, Connector_PinHeader_2.54mm:PinHeader_1x05_P2.54mm_Vertical, symbol PCM_SL_Pin_Headers:PINHD_1x5_Male
- added J7, J9: PINHD_1x9_Male, Connector_PinHeader_2.54mm:PinHeader_1x09_P2.54mm_Vertical, symbol PCM_SL_Pin_Headers:PINHD_1x9_Male
- added J8: PINHD_1x2_Female, Battery:BatteryHolder_MPD_BH-18650-PC2, symbol PCM_SL_Pin_Headers:PINHD_1x2_Female
- added LED1: LED_5mm_RGB_Kcom_BKRG, Connector_PinHeader_2.54mm:PinHeader_1x04_P2.54mm_Vertical, symbol PCM_LED_AKL:LED_5mm_RGB_Kcom_BKRG
- added R1, R2, R3: 330ohm, Resistor_THT:R_Axial_DIN0207_L6.3mm_D2.5mm_P10.16mm_Horizontal, symbol PCM_SL_Resistors:330ohm
- added R10, R4, R5, R6, R8, R9: 4.7k, Resistor_THT:R_Axial_DIN0207_L6.3mm_D2.5mm_P10.16mm_Horizontal, symbol PCM_SL_Resistors:4.7k
- added R11, R12: R_0805 10K, PCM_Resistor_SMD_AKL:R_0805_2012Metric, symbol PCM_Resistor_AKL:R_0805
- added R13, R14, R15, R16, R17, R18, R19, R20, R7: 33ohm, Resistor_THT:R_Axial_DIN0207_L6.3mm_D2.5mm_P10.16mm_Horizontal, symbol PCM_SL_Resistors:33ohm
- added R21: 1k, Resistor_THT:R_Axial_DIN0207_L6.3mm_D2.5mm_P10.16mm_Horizontal, symbol PCM_SL_Resistors:1k
- added SW1, SW2, SW3, SW4: Push_Button, Button_Switch_THT:SW_PUSH_6mm, symbol PCM_SL_Devices:Push_Button
- added U3: AMS1117-3.3, Package_TO_SOT_SMD:SOT-223-3_TabPin2, symbol Regulator_Linear:AMS1117-3.3
- added U4: STM32F103C8Tx, Package_QFP:LQFP-48_7x7mm_P0.5mm, symbol MCU_ST_STM32F1:STM32F103C8Tx
- added Y1: Crystal_8MHz, Crystal:Crystal_HC49-4H_Vertical, symbol PCM_SL_Devices:Crystal_8MHz
- added pot/switch1, pot/switch2: PINHD_1x3_Male, Connector_PinHeader_2.54mm:PinHeader_1x03_P2.54mm_Vertical, symbol PCM_SL_Pin_Headers:PINHD_1x3_Male
- J11, J12, J14: footprint Connector_PinHeader_2.54mm:PinHeader_1x01_P2.54mm_Vertical -> TestPoint:TestPoint_THTPad_2.0x2.0mm_Drill1.0mm
- J4: footprint Connector_PinSocket_2.54mm:PinSocket_1x01_P2.54mm_Vertical -> TestPoint:TestPoint_THTPad_2.0x2.0mm_Drill1.0mm
Connections:
- net Li-ion is gone; now on an unnamed net: D1.2 (A)
- net +3.3V: now also A1.20 (3V3), A1.38 (3V3), C11.1, C12.1, C13.1, C14.1, C4.2, C6.1, C7.1, C8.1, J13.2, J2.1, J6.1, J7.2, J9.2, R12.2, R21.2, SW1.1, SW2.1, SW3.1, SW4.1, U3.2 (VO), U4.24 (VDD), U4.36 (VDD), U4.48 (VDD), U4.9 (VDDA), pot/switch1.1, pot/switch2.1; no longer J12.1
- net BAT-GND: now also J8.2
- net ECL: now also R19.2
- net EDA: now also R20.2
- net Earth: now also A1.19 (GND), A1.39 (GND), A1.40 (GND), C1.1, C10.1, C11.2, C12.2, C13.2, C14.2, C15.2, C2.1, C3.2, C4.1, C6.2, C7.2, C8.2, C9.2, D2.1, J1.2, J13.1, J16.1, J2.2, J6.2, J7.1, J9.1, LED1.2 (A), R10.2, R11.1, R4.2, R5.2, R6.2, R8.1, R9.1, U3.1 (GND), U4.23 (VSS), U4.35 (VSS), U4.47 (VSS), U4.8 (VSSA)
- net INT: now also A1.13 (PB5/MOSI1), U4.41 (PB5)
- net MISO: now also A1.3 (PB14/MISO2), R14.1, U4.27 (PB14); no longer J3.7, U1.7 (MISO)
- net MOSI: now also A1.4 (PB15/MOSI2), R7.1, U4.28 (PB15); no longer J3.4, U1.6 (MOSI)
- net SCL: now also J3.3, A1.30 (SCK1/PA5), R17.1, U4.15 (PA5), U4.42 (PB6)
- net SCLK: now also A1.2 (PB13/SCK2), R15.1, U4.26 (PB13); no longer J3.3, U1.5 (SCK)
- net SDA: now also J3.4, A1.32 (MOSI1/PA7), R18.1, U4.17 (PA7), U4.43 (PB7)
- net VIN: now also C1.2, C2.2, C3.1, U3.3 (VI)
- net +5V: no longer names the net of J11.1
- net A10: no longer names the net of U1.4 (~{CSN})
- net A10: now also R13.2
- net A8 renamed NCS
- net NCS: now also A1.29 (NSS1/PA4), U4.14 (PA4)
- net A9: no longer names the net of U1.3 (CE)
- net A9: now also R16.2
- new net: R8.2, pot/switch2.3
- new net: R9.2, pot/switch1.3
- new net: C9.1, U4.6 (PD1), Y1.1
- new net: LED1.1 (B), R3.2
- new net: LED1.3 (R), R2.1
- new net: LED1.4 (G), R1.2
- new net: D2.2, R21.1
- new net: A1.14 (PB6/SCL1/TX1), R17.2
- new net: A1.15 (PB7/SDA1/RX1), R18.2
- new net: C10.2, U4.5 (PD0), Y1.2
- new net: R15.2, U1.5 (SCK)
- new net: R7.2, U1.6 (MOSI)
- new net: R14.2, U1.7 (MISO)
- new net: R11.2, U4.44 (BOOT0)
- new net 5V: J15.1
- new net AD0: A1.31 (MISO1/PA6), J3.7, U4.16 (PA6)
- new net BATTERY+: J12.1, J8.1
- new net Button1: A1.33 (PB0), J7.6, J9.6, R4.1, SW1.2, U4.18 (PB0)
- new net Button2: A1.34 (PB1), J7.5, J9.5, R5.1, SW2.2, U4.19 (PB1)
- new net Button3: A1.16 (PB8/SCL1), J7.4, J9.4, R6.1, SW3.2, U4.45 (PB8)
- new net Button4: A1.17 (PB9/SDA1), J13.5, J7.3, J9.3, U4.46 (PB9)
- new net Button5: A1.6 (PA9/TX1), J7.9, J9.9, R10.1, SW4.2, U4.21 (PB10)
- new net CE: A1.5 (PA8/CK1), R16.1, U4.29 (PA8)
- new net CSN: A1.1 (PB12/NSS2), R13.1, U4.25 (PB12)
- new net CoinCell: A1.21 (VBAT), J1.1, U4.1 (VBAT)
- new net DRDY: J2.5
- new net LEDB: A1.8 (PA11/~{USB-}), R3.1, U4.32 (PA11)
- new net LEDG: A1.7 (PA10/RX1), R1.1, U4.31 (PA10)
- new net LEDR: A1.35 (SCL2/TX3/PB10), R2.2, U4.30 (PA9)
- new net NRST: C15.1, J6.5, R12.1, U4.7 (NRST)
- new net SCL_M: J2.3, R19.1
- new net SDA_M: J2.4, R20.1
- new net SWCLK: J6.4, U4.37 (PA14)
- new net SWDIO: J6.3, U4.34 (PA13)
- new net TRIG1: A1.27 (TX2/PA2), U4.12 (PA2), pot/switch2.2
- new net TRIG2: A1.28 (RX2/PA3), U4.13 (PA3), pot/switch1.2
- new net X Axis: A1.25 (PA0), J13.3, J7.7, J9.7, U4.10 (PA0)
- new net Z Axis: A1.26 (PA1), J13.4, J7.8, J9.8, U4.11 (PA1)
- no-connect marks 2 -> 1
Other:
- removed sheet Arduino Pro Micro
- removed sheet Level Shifter
- added sheet Connections (Connections.kicad_sch)
- added sheet HID (HID.kicad_sch)
- added sheet Manyometre GY-271 (Manyometre.kicad_sch)
- added sheet ST-LINK Programer (ST-LINK_Programer.kicad_sch)
- added sheet STM32 BluePill F103C8T6_F103C6T6 (STM32BluePillF103C8T6_F103C6T6.kicad_sch)
- added sheet Screew (Screew.kicad_sch)
- added sheet TP4056 Connection (TP4056Connection.kicad_sch)
- added sheet Voltage Regulator (VoltageRegulator.kicad_sch)
- moved on the sheet: D1, J11, J12, J14, J3, J4, U1
